File: Hardware/FEHA-LSC-001-01-Controller-Rev-A/FEHA-LSC-001-01-Controller-Rev-A.kicad_pcb (KiCad board)
At the start: 4 copper layers, 50 x 30 mm, 41 parts, among them CN1 HDGC4001SMD-S-2P, CN2 HDGC4001SMD-S-2P, CN3 USB_DEBUG, Q1 HL2310A, Q2 SI2356DS-T1-GE3, U1 TPS560430XFDBVR, U2 ESP32-C3-MINI-1-H4X(4MB)

Commit message: LSC controller: limits silkscreen, manufacturing files, TVS rationale
- F.SilkS operating limits (CHG-03): 24V DC ONLY, LOAD MAX 1A,
  PSU MAX 30W, USB:24V OFF (1.2 mm bold). DRC unchanged.
- Solder-mask-to-copper clearance 0.005 mm.
- Manufacturing files from the Fabrication Toolkit in production/:
  Gerber/drill zip, BOM, positions, designators, IPC netlist.
- DEC-41: SMBJ26A kept; DEC-10 rationale corrected (clamp above 38 V
  at high pulse current, fails short on an overvoltage supply).
- Spec §0, controller and Hardware READMEs updated.

Co-Authored-By: Claude Opus 5.5 <noreply@anthropic.com>
Other:
- board text added: "24V DC ONLY"
- board text added: "LOAD MAX 1A PSU MAX 30W"
- board text added: "USB:24V OFF"
Changed lines of the file:
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@@
+		)
+	)
+	(gr_text "24V DC\nONLY"
+		(at 101.3272 101.3348 0)
+		(layer "F.SilkS")
+		(effects
+			(font
+				(size 1.2 1.2)
+				(thickness 0.24)
+				(bold yes)
+			)
+			(justify left top)
+		)
+	)
+	(gr_text "USB:24V OFF"
+		(at 132.62 127.3698 0)
+		(layer "F.SilkS")
+		(effects
+			(font
+				(size 1.2 1.2)
+				(thickness 0.24)
+				(bold yes)
+			)
+			(justify left top)
+		)
+	)
+	(gr_text "LOAD MAX 1A\nPSU MAX 30W"
+		(at 135.1854 101.3348 0)
+		(layer "F.SilkS")
+		(effects
+			(font
+				(size 1.2 1.2)
+				(thickness 0.24)
+				(bold yes)
+			)
+			(justify left top)
 		)
 	)
